File: Johnson_Counter.sch (KiCad schematic (older format))
At the start: 32 parts, among them U1 LM555N, U2 4017

Commit message: Add buffer
Parts:
- added BT?: BATTERY, symbol BATTERY
- added U?: CY74FCT827T, MODULE, symbol CY74FCT827T
Connections:
- net +5V: now also U?.24 (VCC)
- net GND: now also BT?.2 (-), U?.1 (~OE1), U?.12 (GND), U?.13 (~OE2)
- net VCC: now also BT?.1 (+)
- net at U2.1 (Q5): now also U?.7 (D5); no longer R4.1
- net at U2.10 (Q4): now also U?.6 (D4); no longer R3.1
- net at U2.11 (Q9): now also U?.11 (D9); no longer R12.2
- net at U2.2 (Q1): now also U?.3 (D1); no longer R9.1
- net at U2.3 (Q0): now also U?.2 (D0); no longer R11.2
- net at U2.4 (Q2): now also U?.4 (D2); no longer R7.1
- net at U2.5 (Q6): now also U?.8 (D6); no longer R6.2
- net at U2.6 (Q7): now also U?.9 (D7); no longer R8.2
- net at U2.7 (Q3): now also U?.5 (D3); no longer R5.1
- net at U2.9 (Q8): now also U?.10 (D8); no longer R10.2
- new net: R5.1, U?.20 (Y3)
- new net: R7.1, U?.21 (Y2)
- new net: R9.1, U?.22 (Y1)
- new net: R6.2, U?.17 (Y6)
- new net: R8.2, U?.16 (Y7)
- new net: R10.2, U?.15 (Y8)
- new net: R12.2, U?.14 (Y9)
- new net: R11.2, U?.23 (Y0)
- new net: R3.1, U?.19 (Y4)
- new net: R4.1, U?.18 (Y5)
Other:
- moved on the sheet: D1, D10, D2, D3, D4, D5, D6, D7, D8, D9, R10, R11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
